Commit message: Add battery & plc communication, 3d lidar localizer & obstacle monitor, and navigation updates

File: my_robot_description/urdf/01-myfirst_backup.urdf (robot description, URDF)
Before this commit: robot my_robot_description, 9 links, 8 joints
Links:
- removed link back_idler
- removed link front_idler
- added link back_left_idler_link, mass 0.5506; collision mesh filename=package://my_robot_description/meshes/back_idler.STL; visual mesh filename=package://my_robot_description/meshes/back_idler.STL
- added link back_right_idler_link, mass 0.5506; collision mesh filename=package://my_robot_description/meshes/back_idler.STL; visual mesh filename=package://my_robot_description/meshes/back_idler.STL
- added link front_left_idler_link, mass 0.5506; collision mesh filename=package://my_robot_description/meshes/front_idler.STL; visual mesh filename=package://my_robot_description/meshes/front_idler.STL
- added link front_right_idler_link, mass 0.5506; collision mesh filename=package://my_robot_description/meshes/front_idler.STL; visual mesh filename=package://my_robot_description/meshes/front_idler.STL
- link back_lidar: mass 0.592505821642753 -> 0.6404
- link base_link: mass 16.5612318297859 -> 63.11417452
- link front_lidar: mass 0.592505826671524 -> 0.6404
- link imu_sensor: mass 0.00312469138199262 -> 0.0031
- link left_wheel: mass 0.629371523823339 -> 2.317732
- link right_wheel: mass 0.629371523823339 -> 2.317732
Joints:
- removed joint backidler
- removed joint frontidler
- added joint back_left_idler: type fixed, parent base_link, child back_left_idler_link, origin xyz=-0.500 0.200 0.071 rpy=0 0 0, axis 0 1 0
- added joint back_right_idler: type fixed, parent base_link, child back_right_idler_link, origin xyz=-0.500 -0.200 0.071 rpy=0 0 0, axis 0 1 0
- added joint front_left_idler: type fixed, parent base_link, child front_left_idler_link, origin xyz=0.500 0.200 0.071 rpy=0 0 0, axis 0 1 0
- added joint front_right_idler: type fixed, parent base_link, child front_right_idler_link, origin xyz=0.500 -0.200 0.071 rpy=0 0 0, axis 0 1 0
- joint backlidar: origin xyz=-0.35538 -0.28336 0.0265 rpy=0 0 -2.3562 -> xyz=-0.690 -0.395 0.1087 rpy=0 0 -2.3562
- joint frontlidar: origin xyz=0.35536 0.28336 0.0265 rpy=0 0 0.7854 -> xyz=0.690 0.395 0.1087 rpy=0 0 0.7854
- joint leftwheel: origin xyz=0 0.2475 0.006 rpy=0 0 0 -> xyz=0 0.300 0.042531 rpy=0 0 0
- joint rightwheel: origin xyz=0 -0.2475 0.006 rpy=0 0 0 -> xyz=0 -0.300 0.042531 rpy=0 0 0
